File: hw/klon_clone.sch (KiCad schematic (older format))
At the start: 72 parts

Commit message: Added power symbols and connectors.
Parts:
- added U? (x2): TL072, symbol Amplifier_Operational:TL072
Other:
- moved on the sheet: C?, R?

Commit message: Schematic wiring done.
Connections:
- net +16V2: now also C?.1, D?.1 (K), U?.8 (V+)
- net +4V5: now also C?.1, R?.1, R?.2, R?.2, R?.2, R?.2, RV?.2, RV?.3, U?.3 (+), U?.5 (+)
- net +9V: now also C?.1, D?.1 (K), D?.2 (A), J?.1, R?.1, R?.2, U?.8 (V+), U?.8 (V+)
- net -8V6: now also C?.1, U?.4 (V-), U?.5 (VOUT)
- net Earth: now also C?.2, C?.2, C?.2, C?.2, C?.2, D?.1 (K), D?.2 (A), D?.2 (A), J?.2, R?.2, R?.2, R?.2, RV?.3, SW?.2 (B), U?.3 (GND), U?.4 (V-)
- net at R?.1: now also C?.2
- net at R?.2: now also J?.T
- net at C?.1: now also R?.1, U?.3 (+)
- net at U?.1: now also C?.1, C?.2, C?.2, R?.1, U?.2 (-)
- net at C?.2: now also C?.1, R?.1, R?.2, RV?.1
- net at C?.1: now also C?.2, R?.2, R?.2
- net at R?.1: now also C?.1, RV?.3, U?.5 (+)
- net at U?.6 (-): now also C?.1, C?.2, R?.1, R?.2
- net at U?.7: now also C?.1, C?.2, R?.1
- net at R?.1: now also RV?.1 (x2)
- net at R?.2: now also C?.2, R?.2
- net at C?.1: now also R?.2 (x2)
- net at R?.1: now also C?.2, D?.1 (K), D?.2 (A), SW?.3 (C)
- net at R?.1: now also C?.1, R?.2
- net at R?.1: now also C?.1, C?.2, R?.1, R?.1, R?.2, U?.2 (-)
- net at SW?.1 (A): now also D?.1 (K)
- net at C?.1: now also C?.1, R?.2
- net at C?.2: now also R?.1 (x3)
- net at R?.2: now also R?.2, R?.2, RV?.2
- net at D?.2 (A): now also R?.1
- net at U?.1: now also C?.1, R?.1, R?.1, R?.2
- net at R?.2: now also RV?.1
- net at R?.1: now also C?.1, R?.2, U?.6 (-)
- net at RV?.2: now also C?.2
- net at RV?.3: now also R?.2
- net at R?.1: now also C?.2, R?.1, U?.7
- net at RV?.2: now also R?.2, SW?.3 (C)
- net at SW?.1 (A): now also R?.1, R?.2
- net at SW?.2 (B): now also J?.T, R?.1, R?.1, R?.1
- net at C?.1: now also R?.1, R?.2
- net at U?.2 (CAP+): now also C?.1, C?.1
- net at U?.4 (CAP-): now also C?.2
- net at D?.1 (K): now also C?.2, D?.2 (A)
- no-connect marks 0 -> 2
Other:
- moved on the sheet: D?, R?, SW?A

Commit message: Component values set.
Parts:
- C? (x2): value C_Small -> 100n
- C? (x2): value C_Small -> 68n
- C?: value C_Small -> 82n
- C?: value C_Small -> 390p
- C? (x7): value C_Small -> 1u
- C?: value C_Small -> 2.2n
- C?: value C_Small -> 390n
- C?: value C_Small -> 27n
- C?: value C_Small -> 820p
- C?: value C_Small -> 3.9n
- C? (x2): value C_Small -> 4.7u
- C? (x2): value C_Small -> 47u
- D? (x2): value D -> 1N34A
- D?: value 1N47xxA -> 1N4742
- R? (x2): value R_Small_US -> 10k
- R?: value R_Small_US -> 1M
- R?: value R_Small_US -> 5.1k
- R?: value R_Small_US -> 422k
- R?: value R_Small_US -> 2k
- R? (x2): value R_Small_US -> 15k
- R? (x2): value R_Small_US -> 1k
- R? (x2): value R_Small_US -> 1.5k
- R?: value R_Small_US -> 22k
- R?: value R_Small_US -> 47k
- R? (x3): value R_Small_US -> 27k
- R?: value R_Small_US -> 12k
- R?: value R_Small_US -> 3.9k
- R?: value R_Small_US -> 392k
- R?: value R_Small_US -> 1.8k
- R? (x4): value R_Small_US -> 100k
- R?: value R_Small_US -> 4.7k
- R? (x2): value R_Small_US -> 560
- R? (x2): value R_Small_US -> 68k
- RV? (x2): value R_POT_US -> 100k
- RV? (x2): value R_POT_US -> 10k
Connections:
- net Earth: now also J?.G, J?.G, J?.S, J?.S
Other:
- moved on the sheet: D?
